File: ortho practice.kicad_pcb (KiCad board)
At the start: 2 copper layers, 233 x 131 mm, 130 parts, among them K1 KEYSW, K10 KEYSW, K11 KEYSW, K12 KEYSW, K13 KEYSW, K14 KEYSW, K15 KEYSW, K16 KEYSW, K17 KEYSW, K18 KEYSW, K19 KEYSW, K2 KEYSW, K20 KEYSW, K21 KEYSW, K22 KEYSW, K23 KEYSW, K24 KEYSW, K25 KEYSW, K26 KEYSW, K27 KEYSW, K28 KEYSW, K29 KEYSW, K3 KEYSW, K30 KEYSW, K31 KEYSW, K32 KEYSW, K33 KEYSW, K34 KEYSW, K35 KEYSW, K36 KEYSW, K37 KEYSW, K38 KEYSW, K39 KEYSW, K4 KEYSW, K40 KEYSW, K41 KEYSW, K42 KEYSW, K43 KEYSW, K44 KEYSW, K45 KEYSW, K46 KEYSW, K47 KEYSW, K48 KEYSW, K49 KEYSW, K5 KEYSW, K50 KEYSW, K51 KEYSW, K52 KEYSW, K53 KEYSW, K54 KEYSW, K55 KEYSW, K56 KEYSW, K57 KEYSW, K58 KEYSW, K59 KEYSW, K6 KEYSW, K60 KEYSW, K7 KEYSW, K8 KEYSW, K9 KEYSW, U1 ProMicro

Commit message: Add files via upload
Parts:
- U1: footprint keebs:Pro_Micro -> promicro:ProMicro
Routing:
- net /col5: track 175.2 -> 151.0 mm
- net /col6: track 189.5 -> 171.5 mm
- net /col12: track 290.1 -> 304.1 mm
- net /col7: track 205.0 -> 192.5 mm
- net /col11: track 269.1 -> 278.4 mm
- net /col8: track 225.6 -> 217.8 mm
- net /col10: track 253.9 -> 257.8 mm
- net /col9: track 239.5 -> 237.8 mm
Other:
- board text added: "B1"
- board text added: "B2"
- board text added: "B3"
- board text added: "B4"
- board text added: "B5"
- board text added: "B6"
- board text added: "C6"
- board text added: "D0"
- board text added: "D1"
- board text added: "D2"
- board text added: "D3"
- board text added: "D4"
- board text added: "D7"
- board text added: "E6"
- board text added: "F4"
- board text added: "F5"
- board text added: "F6"
- board text added: "F7"
- board text added: "GND"
- board text added: "RAW"
- board text added: "RST"
- board text added: "VCC"
- board text added: "d3vastat0r v2.0"
- board text removed: "TX0"
- board text removed: "d3vastat0r v1.0"
