File: ortho practice.sch (KiCad schematic (older format))
At the start: 130 parts, among them K1 KEYSW, K10 KEYSW, K11 KEYSW, K12 KEYSW, K13 KEYSW, K14 KEYSW, K15 KEYSW, K16 KEYSW, K17 KEYSW, K18 KEYSW, K19 KEYSW, K2 KEYSW, K20 KEYSW, K21 KEYSW, K22 KEYSW, K23 KEYSW, K24 KEYSW, K25 KEYSW, K26 KEYSW, K27 KEYSW, K28 KEYSW, K29 KEYSW, K3 KEYSW, K30 KEYSW, K31 KEYSW, K32 KEYSW, K33 KEYSW, K34 KEYSW, K35 KEYSW, K36 KEYSW, K37 KEYSW, K38 KEYSW, K39 KEYSW, K4 KEYSW, K40 KEYSW, K41 KEYSW, K42 KEYSW, K43 KEYSW, K44 KEYSW, K45 KEYSW, K46 KEYSW, K47 KEYSW, K48 KEYSW, K49 KEYSW, K5 KEYSW, K50 KEYSW, K51 KEYSW, K52 KEYSW, K53 KEYSW, K54 KEYSW, K55 KEYSW, K56 KEYSW, K57 KEYSW, K58 KEYSW, K59 KEYSW, K6 KEYSW, K60 KEYSW, K7 KEYSW, K8 KEYSW, K9 KEYSW, U1 ProMicro

Commit message: Add files via upload
Parts:
- U1: footprint keebs:Pro_Micro -> promicro:ProMicro
Changed lines of the file:
@@
 EESchema Schematic File Version 4
-LIBS:ortho practice-cache
 EELAYER 29 0
 EELAYER END
@@
 F 0 "U1" H 9050 6987 60  0000 C CNN
 F 1 "ProMicro" H 9050 6881 60  0000 C CNN
-F 2 "keebs:Pro_Micro" H 9150 4900 60  0001 C CNN
+F 2 "promicro:ProMicro" H 9150 4900 60  0001 C CNN
 F 3 "" H 9150 4900 60  0000 C CNN
 	1    9050 5950
